File: IoTLynx.kicad_sch (KiCad schematic)
At the start: 28 parts, among them J1 USB_C_Receptacle_USB2.0_16P, J2 Conn_01x14, J3 Conn_01x14, U1 ESP32-C6-MINI-1/U, U2 LM1117MP-3.3

Commit message: added some images and files v2
Other:
- company: (none) -> hussamtalkstech.com
- title: (none) -> IoTLynx ESP32-C6 Development board
Changed lines of the file:
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@@
 	(generator_version "9.0")
 	(paper "A4")
+	(title_block
+		(title "IoTLynx ESP32-C6 Development board")
+		(date "2026-01-02")
+		(rev "v0.1")
+		(company "hussamtalkstech.com")
+		(comment 1 "Author: Hussam Al-Hertani")
+	)
 	(rectangle
 		(start 12.7 165.1)
